Commit message: fix: orientation message. progress: leg calibration.

File: champ/src/test_config/urdf/quadruped.urdf (robot description, URDF)
Before this commit: robot quadruped, 21 links, 20 joints
Links:
- link base_link: geometry visual mesh filename=package://test_config/meshes/body-bottom.stl scale=0.0015 0.0015 0.0015
- link lf_hip_link: geometry visual mesh filename=package://test_config/meshes/shoulder-joint-left.stl scale=0.0015 0.0015 0.0015
Joints:
- joint lf_lower_leg_joint: limit lower=-3.14159265359 upper=3.14159265359 effort=25 velocity=1.5 -> lower=-1.57079632679 upper=-1.57079632679 effort=25 velocity=1.5
- joint lh_lower_leg_joint: limit lower=-3.14159265359 upper=3.14159265359 effort=25 velocity=1.5 -> lower=-1.57079632679 upper=-1.57079632679 effort=25 velocity=1.5
- joint rf_lower_leg_joint: limit lower=-3.14159265359 upper=3.14159265359 effort=25 velocity=1.5 -> lower=-1.57079632679 upper=-1.57079632679 effort=25 velocity=1.5
- joint rh_lower_leg_joint: limit lower=-3.14159265359 upper=3.14159265359 effort=25 velocity=1.5 -> lower=-1.57079632679 upper=-1.57079632679 effort=25 velocity=1.5
