Commit message: feat: create quadruped.urdf.xacro and update blender files

File: champ/src/test_config/urdf/quadruped.urdf.xacro (robot description, xacro)
@@ -1,169 +1,497 @@
 <?xml version="1.0" ?>
-<robot name="quadruped"
-    xmlns:xacro="http://www.ros.org/wiki/xacro">
+<robot name="quadruped" xmlns:xacro="http://www.ros.org/wiki/xacro">
     <link name="base_link">
-      <visual>
-        <geometry>
-          <!-- <cylinder length="0.1" radius="0.2"/> -->
-            <mesh
-                filename="package://test_config/meshes/body-bottom.stl"
-                scale="0.0015 0.0015 0.0015"
-            />
-        </geometry>
-      </visual>
-    </link>
-    <link name="lf_hip_debug_link"/>
+        <visual>
+            <origin xyz="0 0 0" rpy="0 0 0"/>
+            <geometry>
+                <mesh
+                    filename="package://test_config/meshes/base.stl"
+                    scale="0.001 0.001 0.001"
+                />
+            </geometry>
+        </visual>
+        <collision>
+            <origin xyz="0 0 0" rpy="0 0 0"/>
+            <geometry>
+                <mesh
+                    filename="package://test_config/meshes/base.stl"
+                    scale="0.001 0.001 0.001"
+                />
+            </geometry>
+        </collision>
+    </link>
+    <link name="f_bumper_link">
+        <visual>
+            <origin xyz="0 0 0" rpy="0 0 0"/>
+            <geometry>
+                <mesh
+                    filename="package://test_config/meshes/bumper.stl"
+                    scale="0.001 0.001 0.001"
+                />
+            </geometry>
+        </visual>
+        <collision>
+            <origin xyz="0 0 0" rpy="0 0 0"/>
+            <geometry>
+                <mesh
+                    filename="package://test_config/meshes/bumper.stl"
+                    scale="0.001 0.001 0.001"
+                />
+            </geometry>
+        </collision>
+    </link>
+    <link name="h_bumper_link">
+        <visual>
+            <origin xyz="0 0 0" rpy="0 0 3.1415"/>
+            <geometry>
+                <mesh
+                    filename="package://test_config/meshes/bumper.stl"
+                    scale="0.001 0.001 0.001"
+                />
+            </geometry>
+        </visual>
+        <collision>
+            <origin xyz="0 0 0" rpy="0 0 3.1415"/>
+            <geometry>
+                <mesh
+                    filename="package://test_config/meshes/bumper.stl"
+                    scale="0.001 0.001 0.001"
+                />
+            </geometry>
+        </collision>
+    </link>
     <link name="lf_hip_link">
-    <visual>
-        <geometry>
-        <mesh
-            filename="package://test_config/meshes/shoulder-joint-left.stl"
-            scale="0.0015 0.0015 0.0015"
-            />
-            </geometry>
-      </visual>
+        <visual>
+            <origin xyz="0 0 0" rpy="0 0 0"/>
+            <geometry>
+                <mesh
+                    filename="package://test_config/meshes/hip.stl"
+                    scale="0.001 0.001 0.001"
+                />
+            </geometry>
+        </visual>
+        <collision>
+            <origin xyz="0 0 0" rpy="0 0 0"/>
+            <geometry>
+                <mesh
+                    filename="package://test_config/meshes/hip.stl"
+                    scale="0.001 0.001 0.001"
+                />
+            </geometry>
+        </collision>
     </link>
     <link name="lf_upper_leg_link">
-    </link>
-    <link name="lf_lower_leg_link"/>
-    <link name="lf_foot_link"/>
-    <link name="rf_hip_debug_link"/>
-    <link name="rf_hip_link"/>
-    <link name="rf_upper_leg_link"/>
-    <link name="rf_lower_leg_link"/>
-    <link name="rf_foot_link"/>
-    <link name="lh_hip_debug_link"/>
-    <link name="lh_hip_link"/>
-    <link name="lh_upper_leg_link"/>
-    <link name="lh_lower_leg_link"/>
-    <link name="lh_foot_link"/>
-    <link name="rh_hip_debug_link"/>
-    <link name="rh_hip_link"/>
-    <link name="rh_upper_leg_link"/>
-    <link name="rh_lower_leg_link"/>
-    <link name="rh_foot_link"/>
-    <joint name="lf_debug_joint" type="fixed">
-        <parent link="base_link"/>
-        <child link="lf_hip_debug_link"/>
-        <origin rpy="0 0 0" xyz="0.1375 0.07 0"/>
+        <visual>
+            <origin xyz="0 0 0" rpy="1.5707 0 3.1415"/>
+            <geometry>
+                <mesh
+                    filename="package://test_config/meshes/upper-leg.stl"
+                    scale="0.001 0.001 0.001"
+                />
+            </geometry>
+        </visual>
+        <collision>
+            <origin xyz="0 0 0" rpy="1.5707 0 3.1415"/>
+            <geometry>
+                <mesh
+                    filename="package://test_config/meshes/upper-leg.stl"
+                    scale="0.001 0.001 0.001"
+                />
+            </geometry>
+        </collision>
+    </link>
+    <link name="lf_lower_leg_link">
+        <visual>
+            <origin xyz="0 0 0" rpy="1.5707 4.7123 0"/>
+            <geometry>
+                <mesh
+                    filename="package://test_config/meshes/lower-leg.stl"
+                    scale="0.001 0.001 0.001"
+                />
+            </geometry>
+        </visual>
+        <collision>
+            <origin xyz="0 0 0" rpy="1.5707 4.7123 0"/>
+            <geometry>
+                <mesh
+                    filename="package://test_config/meshes/lower-leg.stl"
+                    scale="0.001 0.001 0.001"
+                />
+            </geometry>
+        </collision>
+    </link>
+    <link name="lf_foot_link">
+        <visual>
+            <origin xyz="0 0 0" rpy="1.5707 4.7123 0"/>
+            <geometry>
+                <mesh
+                    filename="package://test_config/meshes/foot.stl"
+                    scale="0.001 0.001 0.001"
+                />
+            </geometry>
+        </visual>
+        <collision>
+            <origin xyz="0 0 0" rpy="1.5707 4.7123 0"/>
+            <geometry>
+                <mesh
+                    filename="package://test_config/meshes/foot.stl"
+                    scale="0.001 0.001 0.001"
+                />
+            </geometry>
+        </collision>
+    </link>
+    <link name="rf_hip_link">
+        <visual>
+            <origin xyz="0 0 0" rpy="0 0 0"/>
+            <geometry>
+                <mesh
+                    filename="package://test_config/meshes/hip.stl"
+                    scale="0.001 -0.001 0.001"
+                />
+            </geometry>
+        </visual>
+        <collision>
+            <origin xyz="0 0 0" rpy="0 0 0"/>
+            <geometry>
+                <mesh
+                    filename="package://test_config/meshes/hip.stl"
+                    scale="0.001 -0.001 0.001"
+                />
+            </geometry>
+        </collision>
+    </link>
+    <link name="rf_upper_leg_link">
+        <visual>
+            <origin xyz="0 0 0" rpy="4.7123 0 3.1415"/>
+            <geometry>
+                <mesh
+                    filename="package://test_config/meshes/upper-leg.stl"
+                    scale="0.001 -0.001 0.001"
+                />
+            </geometry>
+        </visual>
+        <collision>
+            <origin xyz="0 0 0" rpy="4.7123 0 3.1415"/>
+            <geometry>
+                <mesh
+                    filename="package://test_config/meshes/upper-leg.stl"
+                    scale="0.001 -0.001 0.001"
+                />
+            </geometry>
+        </collision>
+    </link>
+    <link name="rf_lower_leg_link">
+        <visual>
+            <origin xyz="0 0 0" rpy="4.7123 4.7123 0"/>
+            <geometry>
+                <mesh
+                    filename="package://test_config/meshes/lower-leg.stl"
+                    scale="0.001 -0.001 0.001"
+                />
+            </geometry>
+        </visual>
+        <collision>
+            <origin xyz="0 0 0" rpy="4.7123 4.7123 0"/>
+            <geometry>
+                <mesh
+                    filename="package://test_config/meshes/lower-leg.stl"
+                    scale="0.001 -0.001 0.001"
+                />
+            </geometry>
+        </collision>
+    </link>
+    <link name="rf_foot_link">
+        <visual>
+            <origin xyz="0 0 0" rpy="4.7123 4.7123 0"/>
+            <geometry>
+                <mesh
+                    filename="package://test_config/meshes/foot.stl"
+                    scale="0.001 -0.001 0.001"
+                />
+            </geometry>
+        </visual>
+        <collision>
+            <origin xyz="0 0 0" rpy="4.7123 4.7123 0"/>
+            <geometry>
+                <mesh
+                    filename="package://test_config/meshes/foot.stl"
+                    scale="0.001 -0.001 0.001"
+                />
+            </geometry>
+        </collision>
+    </link>
+    <link name="lh_hip_link">
+        <visual>
+            <origin xyz="0 0 0" rpy="0 0 0"/>
+            <geometry>
+                <mesh
+                    filename="package://test_config/meshes/hip.stl"
+                    scale="-0.001 0.001 0.001"
+                />
+            </geometry>
+        </visual>
+        <collision>
+            <origin xyz="0 0 0" rpy="0 0 0"/>
+            <geometry>
+                <mesh
+                    filename="package://test_config/meshes/hip.stl"
+                    scale="-0.001 0.001 0.001"
+                />
+            </geometry>
+        </collision>
+    </link>
+    <link name="lh_upper_leg_link">
+        <visual>
+            <origin xyz="0 0 0" rpy="1.5707 0 3.1415"/>
+            <geometry>
+                <mesh
+                    filename="package://test_config/meshes/upper-leg.stl"
+                    scale="0.001 0.001 0.001"
+                />
+            </geometry>
+        </visual>
+        <collision>
+            <origin xyz="0 0 0" rpy="1.5707 0 3.1415"/>
+            <geometry>
+                <mesh
+                    filename="package://test_config/meshes/upper-leg.stl"
+                    scale="0.001 0.001 0.001"
+                />
+            </geometry>
+        </collision>
+    </link>
+    <link name="lh_lower_leg_link">
+        <visual>
+            <origin xyz="0 0 0" rpy="1.5707 4.7123 0"/>
+            <geometry>
+                <mesh
+                    filename="package://test_config/meshes/lower-leg.stl"
+                    scale="0.001 0.001 0.001"
+                />
+            </geometry>
+        </visual>
+        <collision>
+            <origin xyz="0 0 0" rpy="1.5707 4.7123 0"/>
+            <geometry>
+                <mesh
+                    filename="package://test_config/meshes/lower-leg.stl"
+                    scale="0.001 0.001 0.001"
+                />
+            </geometry>
+        </collision>
+    </link>
+    <link name="lh_foot_link">
+        <visual>
+            <origin xyz="0 0 0" rpy="1.5707 4.7123 0"/>
+            <geometry>
+                <mesh
+                    filename="package://test_config/meshes/foot.stl"
+                    scale="0.001 0.001 0.001"
+                />
+            </geometry>
+        </visual>
+        <collision>
+            <origin xyz="0 0 0" rpy="1.5707 4.7123 0"/>
+            <geometry>
+                <mesh
+                    filename="package://test_config/meshes/foot.stl"
+                    scale="0.001 0.001 0.001"
+                />
+            </geometry>
+        </collision>
+    </link>
+    <link name="rh_hip_link">
+        <visual>
+            <origin xyz="0 0 0" rpy="0 0 0"/>
+            <geometry>
+                <mesh
+                    filename="package://test_config/meshes/hip.stl"
+                    scale="-0.001 -0.001 0.001"
+                />
+            </geometry>
+        </visual>
+        <collision>
+            <origin xyz="0 0 0" rpy="0 0 0"/>
+            <geometry>
+                <mesh
+                    filename="package://test_config/meshes/hip.stl"
+                    scale="-0.001 -0.001 0.001"
+                />
+            </geometry>
+        </collision>
+    </link>
+    <link name="rh_upper_leg_link">
+        <visual>
+            <origin xyz="0 0 0" rpy="4.7123 0 3.1415"/>
+            <geometry>
+                <mesh
+                    filename="package://test_config/meshes/upper-leg.stl"
+                    scale="0.001 -0.001 0.001"
+                />
+            </geometry>
+        </visual>
+        <collision>
+            <origin xyz="0 0 0" rpy="4.7123 0 3.1415"/>
+            <geometry>
+                <mesh
+                    filename="package://test_config/meshes/upper-leg.stl"
+                    scale="0.001 -0.001 0.001"
+                />
+            </geometry>
+        </collision>
+    </link>
+    <link name="rh_lower_leg_link">
+        <visual>
+            <origin xyz="0 0 0" rpy="4.7123 4.7123 0"/>
+            <geometry>
+                <mesh
+                    filename="package://test_config/meshes/lower-leg.stl"
+                    scale="0.001 -0.001 0.001"
+                />
+            </geometry>
+        </visual>
+        <collision>
+            <origin xyz="0 0 0" rpy="4.7123 4.7123 0"/>
+            <geometry>
+                <mesh
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
Commit message: feat: update joint positions in urdf

File: champ/src/test_config/urdf/quadruped.urdf.xacro (robot description, xacro)
@@ -103,14 +103,14 @@
     <link name="lf_lower_leg_link">
         <visual>
-            <origin xyz="0 0 0" rpy="1.5707 4.7123 0"/>
-            <geometry>
-                <mesh
-                    filename="package://test_config/meshes/lower-leg.stl"
-                    scale="0.001 0.001 0.001"
-                />
-            </geometry>
-        </visual>
-        <collision>
-            <origin xyz="0 0 0" rpy="1.5707 4.7123 0"/>
+            <origin xyz="0 0 0" rpy="1.5707 0 0"/>
+            <geometry>
+                <mesh
+                    filename="package://test_config/meshes/lower-leg.stl"
+                    scale="0.001 0.001 0.001"
+                />
+            </geometry>
+        </visual>
+        <collision>
+            <origin xyz="0 0 0" rpy="1.5707 0 0"/>
             <geometry>
                 <mesh
@@ -123,14 +123,14 @@
     <link name="lf_foot_link">
         <visual>
-            <origin xyz="0 0 0" rpy="1.5707 4.7123 0"/>
-            <geometry>
-                <mesh
-                    filename="package://test_config/meshes/foot.stl"
-                    scale="0.001 0.001 0.001"
-                />
-            </geometry>
-        </visual>
-        <collision>
-            <origin xyz="0 0 0" rpy="1.5707 4.7123 0"/>
+            <origin xyz="0 0 0" rpy="1.5707 0 0"/>
+            <geometry>
+                <mesh
+                    filename="package://test_config/meshes/foot.stl"
+                    scale="0.001 0.001 0.001"
+                />
+            </geometry>
+        </visual>
+        <collision>
+            <origin xyz="0 0 0" rpy="1.5707 0 0"/>
             <geometry>
                 <mesh
@@ -183,14 +183,14 @@
     <link name="rf_lower_leg_link">
         <visual>
-            <origin xyz="0 0 0" rpy="4.7123 4.7123 0"/>
-            <geometry>
-                <mesh
-                    filename="package://test_config/meshes/lower-leg.stl"
-                    scale="0.001 -0.001 0.001"
-                />
-            </geometry>
-        </visual>
-        <collision>
-            <origin xyz="0 0 0" rpy="4.7123 4.7123 0"/>
+            <origin xyz="0 0 0" rpy="4.7123 0 0"/>
+            <geometry>
+                <mesh
+                    filename="package://test_config/meshes/lower-leg.stl"
+                    scale="0.001 -0.001 0.001"
+                />
+            </geometry>
+        </visual>
+        <collision>
+            <origin xyz="0 0 0" rpy="4.7123 0 0"/>
             <geometry>
                 <mesh
@@ -203,14 +203,14 @@
     <link name="rf_foot_link">
         <visual>
-            <origin xyz="0 0 0" rpy="4.7123 4.7123 0"/>
-            <geometry>
-                <mesh
-                    filename="package://test_config/meshes/foot.stl"
-                    scale="0.001 -0.001 0.001"
-                />
-            </geometry>
-        </visual>
-        <collision>
-            <origin xyz="0 0 0" rpy="4.7123 4.7123 0"/>
+            <origin xyz="0 0 0" rpy="4.7123 0 0"/>
+            <geometry>
+                <mesh
+                    filename="package://test_config/meshes/foot.stl"
+                    scale="0.001 -0.001 0.001"
+                />
+            </geometry>
+        </visual>
+        <collision>
+            <origin xyz="0 0 0" rpy="4.7123 0 0"/>
             <geometry>
                 <mesh
@@ -263,14 +263,14 @@
     <link name="lh_lower_leg_link">
         <visual>
-            <origin xyz="0 0 0" rpy="1.5707 4.7123 0"/>
-            <geometry>
-                <mesh
-                    filename="package://test_config/meshes/lower-leg.stl"
-                    scale="0.001 0.001 0.001"
-                />
-            </geometry>
-        </visual>
-        <collision>
-            <origin xyz="0 0 0" rpy="1.5707 4.7123 0"/>
+            <origin xyz="0 0 0" rpy="1.5707 0 0"/>
+            <geometry>
+                <mesh
+                    filename="package://test_config/meshes/lower-leg.stl"
+                    scale="0.001 0.001 0.001"
+                />
+            </geometry>
+        </visual>
+        <collision>
+            <origin xyz="0 0 0" rpy="1.5707 0 0"/>
             <geometry>
                 <mesh
@@ -283,14 +283,14 @@
     <link name="lh_foot_link">
         <visual>
-            <origin xyz="0 0 0" rpy="1.5707 4.7123 0"/>
-            <geometry>
-                <mesh
-                    filename="package://test_config/meshes/foot.stl"
-                    scale="0.001 0.001 0.001"
-                />
-            </geometry>
-        </visual>
-        <collision>
-            <origin xyz="0 0 0" rpy="1.5707 4.7123 0"/>
+            <origin xyz="0 0 0" rpy="1.5707 0 0"/>
+            <geometry>
+                <mesh
+                    filename="package://test_config/meshes/foot.stl"
+                    scale="0.001 0.001 0.001"
+                />
+            </geometry>
+        </visual>
+        <collision>
+            <origin xyz="0 0 0" rpy="1.5707 0 0"/>
             <geometry>
                 <mesh
@@ -343,14 +343,14 @@
     <link name="rh_lower_leg_link">
         <visual>
-            <origin xyz="0 0 0" rpy="4.7123 4.7123 0"/>
-            <geometry>
-                <mesh
-                    filename="package://test_config/meshes/lower-leg.stl"
-                    scale="0.001 -0.001 0.001"
-                />
-            </geometry>
-        </visual>
-        <collision>
-            <origin xyz="0 0 0" rpy="4.7123 4.7123 0"/>
+            <origin xyz="0 0 0" rpy="4.7123 0 0"/>
+            <geometry>
+                <mesh
+                    filename="package://test_config/meshes/lower-leg.stl"
+                    scale="0.001 -0.001 0.001"
+                />
+            </geometry>
+        </visual>
+        <collision>
+            <origin xyz="0 0 0" rpy="4.7123 0 0"/>
             <geometry>
                 <mesh
@@ -363,14 +363,14 @@
     <link name="rh_foot_link">
         <visual>
-            <origin xyz="0 0 0" rpy="4.7123 4.7123 0"/>
-            <geometry>
-                <mesh
-                    filename="package://test_config/meshes/foot.stl"
-                    scale="0.001 -0.001 0.001"
-                />
-            </geometry>
-        </visual>
-        <collision>
-            <origin xyz="0 0 0" rpy="4.7123 4.7123 0"/>
+            <origin xyz="0 0 0" rpy="4.7123 0 0"/>
+            <geometry>
+                <mesh
+                    filename="package://test_config/meshes/foot.stl"
+                    scale="0.001 -0.001 0.001"
+                />
+            </geometry>
+        </visual>
+        <collision>
+            <origin xyz="0 0 0" rpy="4.7123 0 0"/>
             <geometry>
                 <mesh
@@ -413,5 +413,5 @@
     </joint>
     <joint name="lf_foot_joint" type="fixed">
-        <origin xyz="0.1049 0.0002 -0.0093" rpy="0 0 0"/>
+        <origin xyz="-0.0093 -0.0003 -0.1060" rpy="0 0 0"/>
         <parent link="lf_lower_leg_link"/>
         <child link="lf_foot_link"/>
@@ -439,5 +439,5 @@
     </joint>
     <joint name="rf_foot_joint" type="fixed">
-        <origin xyz="0.1049 -0.0002 -0.0093" rpy="0 0 0"/>
+        <origin xyz="-0.0093 -0.0003 -0.1060" rpy="0 0 0"/>
         <parent link="rf_lower_leg_link"/>
         <child link="rf_foot_link"/>
@@ -465,5 +465,5 @@
     </joint>
     <joint name="lh_foot_joint" type="fixed">
-        <origin xyz="0.1049 0.0002 -0.0093" rpy="0 0 0"/>
+        <origin xyz="-0.0093 -0.0003 -0.1060" rpy="0 0 0"/>
         <parent link="lh_lower_leg_link"/>
         <child link="lh_foot_link"/>
@@ -491,5 +491,5 @@
     </joint>
     <joint name="rh_foot_joint" type="fixed">
-        <origin xyz="0.1049 -0.0002 -0.0093" rpy="0 0 0"/>
+        <origin xyz="-0.0093 -0.0003 -0.1060" rpy="0 0 0"/>
         <parent link="rh_lower_leg_link"/>
         <child link="rh_foot_link"/>
