Commit message: feat: update joints' constraints and configurations

File: champ/src/test_config/urdf/quadruped.urdf.xacro (robot description, xacro)
@@ -396,5 +396,5 @@
         <child link="lf_hip_link"/>
         <axis xyz="1 0 0"/>
-        <limit lower="-1.57079632679" upper="1.57079632679" effort="25" velocity="1.5"/>
+        <limit lower="-0.8726" upper="0.8726" effort="25" velocity="1.5"/>
     </joint>
     <joint name="lf_upper_leg_joint" type="revolute">
@@ -403,5 +403,5 @@
         <child link="lf_upper_leg_link"/>
         <axis xyz="0 1 0"/>
-        <limit lower="-1.57079632679" upper="1.57079632679" effort="25" velocity="1.5"/>
+        <limit lower="-2.4434" upper="2.4434" effort="25" velocity="1.5"/>
     </joint>
     <joint name="lf_lower_leg_joint" type="revolute">
@@ -410,5 +410,5 @@
         <child link="lf_lower_leg_link"/>
         <axis xyz="0 1 0"/>
-        <limit lower="-1.57079632679" upper="1.57079632679" effort="25" velocity="1.5"/>
+        <limit lower="-2.0944" upper="-1.0472" effort="25" velocity="1.5"/>
     </joint>
     <joint name="lf_foot_joint" type="fixed">
@@ -422,5 +422,5 @@
         <child link="rf_hip_link"/>
         <axis xyz="1 0 0"/>
-        <limit lower="-1.57079632679" upper="1.57079632679" effort="25" velocity="1.5"/>
+        <limit lower="-0.8726" upper="0.8726" effort="25" velocity="1.5"/>
     </joint>
     <joint name="rf_upper_leg_joint" type="revolute">
@@ -429,5 +429,5 @@
         <child link="rf_upper_leg_link"/>
         <axis xyz="0 1 0"/>
-        <limit lower="-1.57079632679" upper="1.57079632679" effort="25" velocity="1.5"/>
+        <limit lower="-2.4434" upper="2.4434" effort="25" velocity="1.5"/>
     </joint>
     <joint name="rf_lower_leg_joint" type="revolute">
@@ -436,5 +436,5 @@
         <child link="rf_lower_leg_link"/>
         <axis xyz="0 1 0"/>
-        <limit lower="-1.57079632679" upper="1.57079632679" effort="25" velocity="1.5"/>
+        <limit lower="-2.0944" upper="-1.0472" effort="25" velocity="1.5"/>
     </joint>
     <joint name="rf_foot_joint" type="fixed">
@@ -448,5 +448,5 @@
         <child link="lh_hip_link"/>
         <axis xyz="1 0 0"/>
-        <limit lower="-1.57079632679" upper="1.57079632679" effort="25" velocity="1.5"/>
+        <limit lower="-0.8726" upper="0.8726" effort="25" velocity="1.5"/>
     </joint>
     <joint name="lh_upper_leg_joint" type="revolute">
@@ -455,5 +455,5 @@
         <child link="lh_upper_leg_link"/>
         <axis xyz="0 1 0"/>
-        <limit lower="-1.57079632679" upper="1.57079632679" effort="25" velocity="1.5"/>
+        <limit lower="-2.4434" upper="2.4434" effort="25" velocity="1.5"/>
     </joint>
     <joint name="lh_lower_leg_joint" type="revolute">
@@ -462,5 +462,5 @@
         <child link="lh_lower_leg_link"/>
         <axis xyz="0 1 0"/>
-        <limit lower="-1.57079632679" upper="1.57079632679" effort="25" velocity="1.5"/>
+        <limit lower="-2.0944" upper="-1.0472" effort="25" velocity="1.5"/>
     </joint>
     <joint name="lh_foot_joint" type="fixed">
@@ -474,5 +474,5 @@
         <child link="rh_hip_link"/>
         <axis xyz="1 0 0"/>
-        <limit lower="-1.57079632679" upper="1.57079632679" effort="25" velocity="1.5"/>
+        <limit lower="-0.8726" upper="0.8726" effort="25" velocity="1.5"/>
     </joint>
     <joint name="rh_upper_leg_joint" type="revolute">
@@ -481,5 +481,5 @@
         <child link="rh_upper_leg_link"/>
         <axis xyz="0 1 0"/>
-        <limit lower="-1.57079632679" upper="1.57079632679" effort="25" velocity="1.5"/>
+        <limit lower="-2.4434" upper="2.4434" effort="25" velocity="1.5"/>
     </joint>
     <joint name="rh_lower_leg_joint" type="revolute">
@@ -488,5 +488,5 @@
         <child link="rh_lower_leg_link"/>
         <axis xyz="0 1 0"/>
-        <limit lower="-1.57079632679" upper="1.57079632679" effort="25" velocity="1.5"/>
+        <limit lower="-2.0944" upper="-1.0472" effort="25" velocity="1.5"/>
     </joint>
     <joint name="rh_foot_joint" type="fixed">

Commit message: feat: update urdf file

File: champ/src/test_config/urdf/quadruped.urdf.xacro (robot description, xacro)
@@ -403,5 +403,5 @@
         <child link="lf_upper_leg_link"/>
         <axis xyz="0 1 0"/>
-        <limit lower="-2.4434" upper="2.4434" effort="25" velocity="1.5"/>
+        <limit lower="-1.0472" upper="1.0472" effort="25" velocity="1.5"/>
     </joint>
     <joint name="lf_lower_leg_joint" type="revolute">
@@ -429,5 +429,5 @@
         <child link="rf_upper_leg_link"/>
         <axis xyz="0 1 0"/>
-        <limit lower="-2.4434" upper="2.4434" effort="25" velocity="1.5"/>
+        <limit lower="-1.0472" upper="1.0472" effort="25" velocity="1.5"/>
     </joint>
     <joint name="rf_lower_leg_joint" type="revolute">
@@ -455,5 +455,5 @@
         <child link="lh_upper_leg_link"/>
         <axis xyz="0 1 0"/>
-        <limit lower="-2.4434" upper="2.4434" effort="25" velocity="1.5"/>
+        <limit lower="-1.0472" upper="1.0472" effort="25" velocity="1.5"/>
     </joint>
     <joint name="lh_lower_leg_joint" type="revolute">
@@ -481,5 +481,5 @@
         <child link="rh_upper_leg_link"/>
         <axis xyz="0 1 0"/>
-        <limit lower="-2.4434" upper="2.4434" effort="25" velocity="1.5"/>
+        <limit lower="-1.0472" upper="1.0472" effort="25" velocity="1.5"/>
     </joint>
     <joint name="rh_lower_leg_joint" type="revolute">
