Commit message: fix: change mesh path in urdf

File: test_config/urdf/quadruped.urdf (robot description, URDF)
Before this commit: robot quadruped, 21 links, 20 joints
Links:
- link camera_link: geometry collision box size=0.02505 0.09 0.025; visual mesh filename=package://realsense-ros/realsense2_description/meshes/d435.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
