Commit message: feat: added camera urdf. Modified servo pins.

File: IK_engine/src/test_config/urdf/quadruped.urdf.xacro (robot description, xacro)
@@ -1,4 +1,6 @@
 <?xml version="1.0" ?>
 <robot name="quadruped" xmlns:xacro="http://www.ros.org/wiki/xacro">
+    <xacro:arg name="use_nominal_extrinsics" default="false" />
+     <xacro:include filename="$(find realsense2_description)/urdf/_d435i.urdf.xacro"/>
     <link name="base_link">
         <visual>
@@ -21,4 +23,7 @@
         </collision>
     </link>
+    <xacro:sensor_d435i parent="base_link" use_nominal_extrinsics="$(arg use_nominal_extrinsics)">
+        <origin xyz="0.075 0 0.068" rpy="0 0 0"/>
+    </xacro:sensor_d435i>
     <link name="f_bumper_link">
         <visual>

Commit message: feat: add tower component to urdf

File: IK_engine/src/test_config/urdf/quadruped.urdf.xacro (robot description, xacro)
@@ -23,4 +23,24 @@
         </collision>
     </link>
+    <link name="tower_link">
+        <visual>
+            <origin xyz="0 0 0" rpy="0 0 0"/>
+            <geometry>
+                <mesh
+                    filename="package://test_config/meshes/tower.stl"
+                    scale="0.001 0.001 0.001"
+                />
+            </geometry>
+        </visual>
+        <collision>
+            <origin xyz="0 0 0" rpy="0 0 0"/>
+            <geometry>
+                <mesh
+                    filename="package://test_config/meshes/tower.stl"
+                    scale="0.001 0.001 0.001"
+                />
+            </geometry>
+        </collision>
+    </link>
     <xacro:sensor_d435i parent="base_link" use_nominal_extrinsics="$(arg use_nominal_extrinsics)">
         <origin xyz="0.075 0 0.068" rpy="0 0 0"/>
@@ -386,4 +406,9 @@
         </collision>
     </link>
+    <joint name="tower_joint" type="fixed">
+        <origin xyz="0.0056 0.0068 0.10042" rpy="0 0 0"/>
+        <parent link="base_link"/>
+        <child link="tower_link"/>
+    </joint>
     <joint name="f_bumper_joint" type="fixed">
         <origin xyz="0.1203 0.0000 -0.0042" rpy="0 0 0"/>
