Commit message: feat: generate the urdf file from xacro

File: IK_engine/src/test_config/urdf/quadruped.urdf (robot description, URDF)
Before this commit: robot quadruped, 21 links, 20 joints
Links:
- added link tower_link; collision mesh filename=package://test_config/meshes/tower.stl scale=0.001 0.001 0.001; visual mesh filename=package://test_config/meshes/tower.stl scale=0.001 0.001 0.001
Joints:
- added joint tower_joint: type fixed, parent base_link, child tower_link, origin xyz=0.0056 0.0068 0.10042 rpy=0 0 0
- joint camera_link_joint: origin xyz=0.0106 0.0175 0.0125 rpy=0 0 0 -> xyz=0.010600000000000002 0.0175 0.0125 rpy=0 0 0

Commit message: fix: update z offset of camera_link

File: IK_engine/src/test_config/urdf/quadruped.urdf (robot description, URDF)
Before this commit: robot quadruped, 22 links, 21 joints
Joints:
- joint camera_joint: origin xyz=0.075 0 0.068 rpy=0 0 0 -> xyz=0.075 0 0.099 rpy=0 0 0

File: IK_engine/src/test_config/urdf/quadruped.urdf.xacro (robot description, xacro)
@@ -44,5 +44,5 @@
     </link>
     <xacro:sensor_d435i parent="base_link" use_nominal_extrinsics="$(arg use_nominal_extrinsics)">
-        <origin xyz="0.075 0 0.068" rpy="0 0 0"/>
+        <origin xyz="0.075 0 0.099" rpy="0 0 0"/>
     </xacro:sensor_d435i>
     <link name="f_bumper_link">
